File: support/EAGLE/symbol_reference.sch (EAGLE design)
At the start: 23 parts, among them IC1 TL072P, IC2 TL072P, IC3 A1301UA, M1 SMALL_SERVO, Q1 IRF540, T1 2N3904

Commit message: Updating to upstream: 3pirobot, mobile, Fritzing, exercise changes.
Squashed commit including the following:
  Importing Fritzing resources from 2014 physcomp-examples.
  Adding 7805 to regulator exercise.
  Adding 123D Circuits exercise blank.
  Updated 3pi and mobile exercises
  Additional 3pi exercises.
  Adding 3pi-robot exercises.
Parts:
- added IC4: 7805T, linear:7805T
Changed lines of the file:
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@@
 <part name="S2" library="switch" deviceset="TL36PO" device=""/>
 <part name="U$3" library="SparkFun-Electromechanical" deviceset="RELAY-2" device="G5Q"/>
+<part name="IC4" library="linear" deviceset="78*" device="T" technology="05"/>
 </parts>
 <sheets>
@@
 <instance part="S2" gate="BEF1" x="320.04" y="223.52"/>
 <instance part="U$3" gate="G$1" x="35.56" y="127"/>
+<instance part="IC4" gate="A1" x="60.96" y="81.28"/>
 </instances>
 <busses>
